Commit message: removed plugins from pepper.urdf

File: urdf/pepper.urdf (robot description, URDF)
Before this commit: robot JulietteY20MP, 83 links, 82 joints
Links:
- link Neck: mass 0.27391 -> 0.001
- link RBicep: geometry visual mesh filename=package://pepper_meshes/meshes/1.0/RShoulderRoll.dae scale=0.1 0.1 0.1
- link RForeArm: geometry visual mesh filename=package://pepper_meshes/meshes/1.0/RElbowRoll.dae scale=0.1 0.1 0.1
- link RShoulder: geometry visual mesh filename=package://pepper_meshes/meshes/1.0/RShoulderPitch.dae scale=0.1 0.1 0.1
- link base_link: mass None -> 1.0; geometry collision box size=0.5 0.15 1.5
- link l_wrist: geometry visual mesh filename=package://pepper_meshes/meshes/1.0/LWristYaw.dae scale=0.1 0.1 0.1
- link r_wrist: geometry visual mesh filename=package://pepper_meshes/meshes/1.0/RWristYaw.dae scale=0.1 0.1 0.1
- link torso: mass 3.99533 -> 0.001
Joints:
- joint HeadPitch: type revolute -> fixed
- joint HeadYaw: type revolute -> fixed
- joint HipPitch: type revolute -> fixed
- joint HipRoll: type revolute -> fixed
- joint KneePitch: type revolute -> fixed
- joint LElbowRoll: type revolute -> fixed
- joint LElbowYaw: type revolute -> fixed
- joint LFinger11: type continuous -> fixed
- joint LFinger12: type continuous -> fixed
- joint LFinger13: type continuous -> fixed
- joint LFinger21: type continuous -> fixed
- joint LFinger22: type continuous -> fixed
- joint LFinger23: type continuous -> fixed
- joint LFinger31: type continuous -> fixed
- joint LFinger32: type continuous -> fixed
- joint LFinger33: type continuous -> fixed
- joint LFinger41: type continuous -> fixed
- joint LFinger42: type continuous -> fixed
- joint LFinger43: type continuous -> fixed
- joint LHand: type revolute -> fixed
- joint LShoulderPitch: type revolute -> fixed
- joint LShoulderRoll: type revolute -> fixed
- joint LThumb1: type continuous -> fixed
- joint LThumb2: type continuous -> fixed
- joint LWristYaw: type revolute -> fixed
- joint RElbowRoll: type revolute -> fixed
- joint RElbowYaw: type revolute -> fixed
- joint RFinger11: type continuous -> fixed
- joint RFinger12: type continuous -> fixed
- joint RFinger13: type continuous -> fixed
- joint RFinger21: type continuous -> fixed
- joint RFinger22: type continuous -> fixed
- joint RFinger23: type continuous -> fixed
- joint RFinger31: type continuous -> fixed
- joint RFinger32: type continuous -> fixed
- joint RFinger33: type continuous -> fixed
- joint RFinger41: type continuous -> fixed
- joint RFinger42: type continuous -> fixed
- joint RFinger43: type continuous -> fixed
- joint RHand: type revolute -> fixed
- joint RShoulderPitch: type revolute -> fixed
- joint RShoulderRoll: type revolute -> fixed
- joint RThumb1: type continuous -> fixed
- joint RThumb2: type continuous -> fixed
- joint RWristYaw: type revolute -> fixed
- joint WheelB: type continuous -> fixed
- joint WheelFL: type continuous -> fixed
- joint WheelFR: type continuous -> fixed
