Commit message: Adding Pepper (using Turtle Xacro Structure)!

File: urdf/pepper.urdf.xacro (robot description, xacro)
@@ -1,12 +1,24 @@
 <?xml version="1.0" ?>
-<!-- =================================================================================== -->
-<!-- |    This document was autogenerated by xacro from pepper_robot.xacro             | -->
-<!-- |    EDITING THIS FILE BY HAND IS NOT RECOMMENDED                                 | -->
-<!-- =================================================================================== -->
-<!--******************************************************************
- ****** File automatically generated by generate_urdf.py script ******
- *********************************************************************-->
-<robot name="JulietteY20MP" xmlns:xacro="http://www.ros.org/wiki/xacro">
+<robot name="turtlebot3_pepper_v" xmlns:xacro="http://ros.org/wiki/xacro">
+  <xacro:include filename="$(find turtlebot3_description)/urdf/common_properties.xacro"/>
+  <xacro:include filename="$(find turtlebot3_description)/urdf/turtlebot3_waffle.gazebo.xacro"/>
+  <xacro:property name="r200_cam_rgb_px" value="0.005"/>
+  <xacro:property name="r200_cam_rgb_py" value="0.018"/>
+  <xacro:property name="r200_cam_rgb_pz" value="0.013"/>
+  <xacro:property name="r200_cam_depth_offset" value="0.01"/>
+  <link name="base_footprint"/>
+  <joint name="base_joint" type="fixed">
+    <parent link="base_footprint"/>
+    <child link="base_link" />
+    <origin xyz="0 0 0.010" rpy="0 0 0"/>
+  </joint>
   <link name="base_link">
+    <visual>
+      <origin xyz="-0.064 0 0.45" rpy="0 0 0"/>
+      <geometry>
+        <box size="0.23 0.23 0.8" />
+      </geometry>
+      <material name="light_black"/>
+    </visual>
     <collision>
       <origin xyz="0 0 0.3" />
@@ -16,9 +28,109 @@
     </collision>
     <inertial>
-      <mass value="1.0"/>
+      <origin xyz="0 0 0" rpy="0 0 0"/>
+      <mass value="1.3729096e+00"/>
+      <inertia ixx="8.7002718e-03" ixy="-4.7576583e-05" ixz="1.1160499e-04"
+               iyy="8.6195418e-03" iyz="-3.5422299e-06"
+               izz="1.4612727e-02" />
+    </inertial>
+  </link>
+<!-- Links From Turtle -->
+  <joint name="wheel_left_joint" type="continuous">
+    <parent link="base_link"/>
+    <child link="wheel_left_link"/>
+    <origin xyz="0.0 0.144 0.023" rpy="-1.57 0 0"/>
+    <axis xyz="0 0 1"/>
+  </joint>
+  <link name="wheel_left_link">
+<!--    <visual>-->
+<!--      <origin xyz="0 0 0" rpy="1.57 0 0"/>-->
+<!--      <geometry>-->
+<!--        <mesh filename="package://turtlebot3_description/meshes/wheels/left_tire.stl" scale="0.001 0.001 0.001"/>-->
+<!--      </geometry>-->
+<!--      <material name="dark"/>-->
+<!--    </visual>-->
+    <collision>
+      <origin xyz="0 0 0" rpy="0 0 0"/>
+      <geometry>
+        <cylinder length="0.018" radius="0.033"/>
+      </geometry>
+    </collision>
+    <inertial>
+      <origin xyz="0 0 0" />
+      <mass value="2.8498940e-02" />
+      <inertia ixx="1.1175580e-05" ixy="-4.2369783e-11" ixz="-5.9381719e-09"
+               iyy="1.1192413e-05" iyz="-1.4400107e-11"
+               izz="2.0712558e-05" />
+      </inertial>
+  </link>
+  <joint name="wheel_right_joint" type="continuous">
+    <parent link="base_link"/>
+    <child link="wheel_right_link"/>
+    <origin xyz="0.0 -0.144 0.023" rpy="-1.57 0 0"/>
+    <axis xyz="0 0 1"/>
+  </joint>
+  <link name="wheel_right_link">
+<!--    <visual>-->
+<!--      <origin xyz="0 0 0" rpy="1.57 0 0"/>-->
+<!--      <geometry>-->
+<!--        <mesh filename="package://turtlebot3_description/meshes/wheels/right_tire.stl" scale="0.001 0.001 0.001"/>-->
+<!--      </geometry>-->
+<!--      <material name="dark"/>-->
+<!--    </visual>-->
+    <collision>
+      <origin xyz="0 0 0" rpy="0 0 0"/>
+      <geometry>
+        <cylinder length="0.018" radius="0.033"/>
+      </geometry>
+    </collision>
+    <inertial>
+      <origin xyz="0 0 0" />
+      <mass value="2.8498940e-02" />
+      <inertia ixx="1.1175580e-05" ixy="-4.2369783e-11" ixz="-5.9381719e-09"
+               iyy="1.1192413e-05" iyz="-1.4400107e-11"
+               izz="2.0712558e-05" />
+      </inertial>
+  </link>
+  <joint name="caster_back_right_joint" type="fixed">
+    <parent link="base_link"/>
+    <child link="caster_back_right_link"/>
+    <origin xyz="-0.177 -0.064 -0.004" rpy="-1.57 0 0"/>
+  </joint>
+  <link name="caster_back_right_link">
+    <collision>
+      <origin xyz="0 0.001 0" rpy="0 0 0"/>
+      <geometry>
+        <box size="0.030 0.009 0.020"/>
+      </geometry>
+    </collision>
+    <inertial>
+      <origin xyz="0 0 0" />
+      <mass value="0.005" />
       <inertia ixx="0.001" ixy="0.0" ixz="0.0"
-               iyy="0.001" iyz="0.0" izz="0.001"/> <!-- Inertia tensor -->
-    </inertial>
-  </link>
+               iyy="0.001" iyz="0.0"
+               izz="0.001" />
+    </inertial>
+  </link>
+  <joint name="caster_back_left_joint" type="fixed">
+    <parent link="base_link"/>
+    <child link="caster_back_left_link"/>
+    <origin xyz="-0.177 0.064 -0.004" rpy="-1.57 0 0"/>
+  </joint>
+  <link name="caster_back_left_link">
+    <collision>
+      <origin xyz="0 0.001 0" rpy="0 0 0"/>
+      <geometry>
+        <box size="0.030 0.009 0.020"/>
+      </geometry>
+    </collision>
+    <inertial>
+      <origin xyz="0 0 0" />
+      <mass value="0.005" />
+      <inertia ixx="0.001" ixy="0.0" ixz="0.0"
+               iyy="0.001" iyz="0.0"
+               izz="0.001" />
+    </inertial>
+  </link>
+<!---->
   <joint name="HeadYaw" type="fixed">
     <parent link="torso"/>

Commit message: pepper is now loaded (not moving very good yet!)

File: urdf/pepper.urdf.xacro (robot description, xacro)
@@ -14,15 +14,15 @@
   </joint>
   <link name="base_link">
-    <visual>
-      <origin xyz="-0.064 0 0.45" rpy="0 0 0"/>
-      <geometry>
-        <box size="0.23 0.23 0.8" />
-      </geometry>
-      <material name="light_black"/>
-    </visual>
+<!--    <visual>-->
+<!--      <origin xyz="-0.064 0 0.45" rpy="0 0 0"/>-->
+<!--      <geometry>-->
+<!--        <box size="0.23 0.23 0.8" />-->
+<!--      </geometry>-->
+<!--      <material name="light_black"/>-->
+<!--    </visual>-->
     <collision>
       <origin xyz="0 0 0.3" />
       <geometry>
-        <box size="0.5 0.15 1.5"/>
+        <box size="0.5 0.15 0.2"/>
       </geometry>
     </collision>
@@ -43,11 +43,11 @@
   </joint>
   <link name="wheel_left_link">
-<!--    <visual>-->
-<!--      <origin xyz="0 0 0" rpy="1.57 0 0"/>-->
-<!--      <geometry>-->
-<!--        <mesh filename="package://turtlebot3_description/meshes/wheels/left_tire.stl" scale="0.001 0.001 0.001"/>-->
-<!--      </geometry>-->
-<!--      <material name="dark"/>-->
-<!--    </visual>-->
+    <visual>
+      <origin xyz="0 0 0" rpy="1.57 0 0"/>
+      <geometry>
+        <mesh filename="package://turtlebot3_description/meshes/wheels/left_tire.stl" scale="0.001 0.001 0.001"/>
+      </geometry>
+      <material name="dark"/>
+    </visual>
     <collision>
       <origin xyz="0 0 0" rpy="0 0 0"/>
@@ -71,11 +71,11 @@
   </joint>
   <link name="wheel_right_link">
-<!--    <visual>-->
-<!--      <origin xyz="0 0 0" rpy="1.57 0 0"/>-->
-<!--      <geometry>-->
-<!--        <mesh filename="package://turtlebot3_description/meshes/wheels/right_tire.stl" scale="0.001 0.001 0.001"/>-->
-<!--      </geometry>-->
-<!--      <material name="dark"/>-->
-<!--    </visual>-->
+    <visual>
+      <origin xyz="0 0 0" rpy="1.57 0 0"/>
+      <geometry>
+        <mesh filename="package://turtlebot3_description/meshes/wheels/right_tire.stl" scale="0.001 0.001 0.001"/>
+      </geometry>
+      <material name="dark"/>
+    </visual>
     <collision>
       <origin xyz="0 0 0" rpy="0 0 0"/>
@@ -133,4 +133,29 @@
   </link>
 <!---->
+  <joint name="base_link_fixedjoint" type="fixed">
+    <parent link="base_link"/>
+    <child link="torso"/>
+    <origin rpy="0 0 0" xyz="-0.1 0 0.8"/>
+    <axis xyz="0 0 0"/>
+  </joint>
+  <link name="torso">
+    <inertial>
+      <mass value="0.001"/>
+      <inertia ixx="0.0" ixy="0" ixz="0.0" iyy="0.0" iyz="-0.0" izz="0.0"/>
+      <origin rpy="0 0 0" xyz="0.00322 0 -0.01029"/>
+    </inertial>
+    <visual>
+      <geometry>
+        <mesh filename="package://pepper_meshes/meshes/1.0/Torso.dae" scale="0.1 0.1 0.1"/>
+      </geometry>
+      <origin rpy="0 0 0" xyz="0 0 0"/>
+    </visual>
+    <collision>
+      <geometry>
+        <mesh filename="package://pepper_meshes/meshes/1.0/Torso_0.10.stl" scale="0.1 0.1 0.1"/>
+      </geometry>
+      <origin rpy="0 0 0" xyz="0 0 0"/>
+    </collision>
+  </link>
   <joint name="HeadYaw" type="fixed">
     <parent link="torso"/>
@@ -263,35 +288,10 @@
     </collision>
   </link>
-  <joint name="base_footprint_joint" type="fixed">
-    <parent link="Tibia"/>
-    <child link="base_footprint"/>
-    <origin rpy="0 0 0" xyz="0 0 -0.334"/>
-  </joint>
-  <link name="base_footprint"/>
-  <joint name="base_link_fixedjoint" type="fixed">
-    <parent link="base_link"/>
-    <child link="torso"/>
-    <origin rpy="0 0 0" xyz="0 0 0"/>
-    <axis xyz="0 0 0"/>
-  </joint>
-  <link name="torso">
-    <inertial>
-      <mass value="0.001"/>
-      <inertia ixx="0.0" ixy="0" ixz="0.0" iyy="0.0" iyz="-0.0" izz="0.0"/>
-      <origin rpy="0 0 0" xyz="0.00322 0 -0.01029"/>
-    </inertial>
-    <visual>
-      <geometry>
-        <mesh filename="package://pepper_meshes/meshes/1.0/Torso.dae" scale="0.1 0.1 0.1"/>
-      </geometry>
-      <origin rpy="0 0 0" xyz="0 0 0"/>
-    </visual>
-    <collision>
-      <geometry>
-        <mesh filename="package://pepper_meshes/meshes/1.0/Torso_0.10.stl" scale="0.1 0.1 0.1"/>
-      </geometry>
-      <origin rpy="0 0 0" xyz="0 0 0"/>
-    </collision>
-  </link>
+<!--  <joint name="base_footprint_joint" type="fixed">-->
+<!--    <parent link="Tibia"/>-->
+<!--    <child link="base_footprint"/>-->
+<!--    <origin rpy="0 0 0" xyz="0 0 -0.334"/>-->
+<!--  </joint>-->
+<!--  <link name="base_footprint"/>-->
   <joint name="LShoulderPitch" type="fixed">
     <parent link="torso"/>
@@ -580,225 +580,225 @@
     </inertial>
   </link>
-  <link name="SonarBack_frame"/>
-  <joint name="Sonar/Back_sensor_fixedjoint" type="fixed">
-    <parent link="Tibia"/>
-    <child link="SonarBack_frame"/>
-    <origin rpy="-1.81761e-08 -0.209438 -3.14159" xyz="-0.0718 0 -0.0534"/>
-    <axis xyz="0 0 0"/>
-  </joint>
-  <link name="CameraBottom_optical_frame"/>
-  <joint name="CameraBottom_optical_frame_fixedjoint" type="fixed">
-    <parent link="CameraBottom_frame"/>
-    <child link="CameraBottom_optical_frame"/>
-    <origin rpy="-1.57079632679 0 -1.57079632679" xyz="0 0 0"/>
-  </joint>
-  <link name="CameraDepth_optical_frame"/>
-  <joint name="CameraDepth_optical_frame_fixedjoint" type="fixed">
-    <parent link="CameraDepth_frame"/>
-    <child link="CameraDepth_optical_frame"/>
-    <origin rpy="-1.57079632679 0 -1.57079632679" xyz="0 0 0"/>
-  </joint>
-  <link name="LHandTouchBack_frame"/>
-  <joint name="LHand/Touch/Back_sensor_fixedjoint" type="fixed">
-    <parent link="l_wrist"/>
-    <child link="LHandTouchBack_frame"/>
-    <origin rpy="1.5708 -1.5708 -3.14159" xyz="0.0523 0 0.0304"/>
-    <axis xyz="0 0 0"/>
-  </joint>
-  <link name="VerticalLeftLaser_frame"/>
-  <joint name="LaserSensor/VerticalLeft_sensor_fixedjoint" type="fixed">
-    <parent link="Tibia"/>
-    <child link="VerticalLeftLaser_frame"/>
-    <origin rpy="0 0.349066 0" xyz="0.0562 0 -0.0692"/>
-    <axis xyz="0 0 0"/>
-  </joint>
-  <link name="SurroundingFrontLaser_device_frame"/>
-  <joint name="LaserSensor/Front_sensor_fixedjoint" type="fixed">
-    <parent link="Tibia"/>
-    <child link="SurroundingFrontLaser_device_frame"/>
-    <origin rpy="0 0.349066 0" xyz="0.0562 0 -0.0692"/>
-    <axis xyz="0 0 0"/>
-  </joint>
-  <link name="BumperB_frame"/>
-  <joint name="Bumper/Back_sensor_fixedjoint" type="fixed">
-    <parent link="Tibia"/>
-    <child link="BumperB_frame"/>
-    <origin rpy="0 0 -3.14159" xyz="-0.251 0 -0.264"/>
-    <axis xyz="0 0 0"/>
-  </joint>
-  <link name="SurroundingLeftLaser_frame"/>
-  <joint name="LaserSensor/Left_projected_sensor_fixedjoint" type="fixed">
-    <parent link="Tibia"/>
-    <child link="SurroundingLeftLaser_frame"/>
-    <origin rpy="0 0 1.75728" xyz="-0.018 0.0899 -0.334"/>
-    <axis xyz="0 0 0"/>
-  </joint>
-  <link name="ShovelLaser_frame"/>
-  <joint name="LaserSensor/Shovel_sensor_fixedjoint" type="fixed">
-    <parent link="Tibia"/>
-    <child link="ShovelLaser_frame"/>
-    <origin rpy="0 0.349066 0" xyz="0.0562 0 -0.0692"/>
-    <axis xyz="0 0 0"/>
-  </joint>
-  <link name="ImuTorsoAccelerometer_frame"/>
-  <joint name="Accelerometer_sensor_fixedjoint" type="fixed">
-    <parent link="torso"/>
-    <child link="ImuTorsoAccelerometer_frame"/>
-    <origin rpy="0 0 0" xyz="0.00239 -0.03575 0.00626"/>
-    <axis xyz="0 0 0"/>
-  </joint>
-  <link name="RSpeaker_frame"/>
-  <joint name="SpeakerRight_sensor_fixedjoint" type="fixed">
-    <parent link="Head"/>
-    <child link="RSpeaker_frame"/>
-    <origin rpy="0 0 0" xyz="0 0 0"/>
-    <axis xyz="0 0 0"/>
-  </joint>
-  <link name="SurroundingRightLaser_device_frame"/>
-  <joint name="LaserSensor/Right_sensor_fixedjoint" type="fixed">
-    <parent link="Tibia"/>
-    <child link="SurroundingRightLaser_device_frame"/>
-    <origin rpy="0 0.349066 -1.5708" xyz="-0.018 -0.0899 -0.0759"/>
-    <axis xyz="0 0 0"/>
-  </joint>
-  <link name="LSpeaker_frame"/>
-  <joint name="SpeakerLeft_sensor_fixedjoint" type="fixed">
-    <parent link="Head"/>
-    <child link="LSpeaker_frame"/>
-    <origin rpy="0 0 0" xyz="0 0 0"/>
-    <axis xyz="0 0 0"/>
-  </joint>
-  <link name="RHandTouchBack_frame"/>
-  <joint name="RHand/Touch/Back_sensor_fixedjoint" type="fixed">
-    <parent link="r_wrist"/>
-    <child link="RHandTouchBack_frame"/>
-    <origin rpy="1.5708 -1.5708 -3.14159" xyz="0.0523 0 0.0304"/>
-    <axis xyz="0 0 0"/>
-  </joint>
-  <link name="CameraTop_frame"/>
-  <joint name="CameraTop_sensor_fixedjoint" type="fixed">
-    <parent link="Head"/>
-    <child link="CameraTop_frame"/>
-    <origin rpy="0 0 0" xyz="0.08601 0 0.16284"/>
-    <axis xyz="0 0 0"/>
-  </joint>
-  <link name="SurroundingLeftLaser_device_frame"/>
-  <joint name="LaserSensor/Left_sensor_fixedjoint" type="fixed">
-    <parent link="Tibia"/>
-    <child link="SurroundingLeftLaser_device_frame"/>
-    <origin rpy="0 0.349066 1.5708" xyz="-0.018 0.0899 -0.0759"/>
-    <axis xyz="0 0 0"/>
-  </joint>
-  <link name="CameraDepth_frame"/>
-  <joint name="CameraDepth_sensor_fixedjoint" type="fixed">
-    <parent link="Head"/>
-    <child link="CameraDepth_frame"/>
-    <origin rpy="0 0 0" xyz="0.05138 0.039 0.1194"/>
-    <axis xyz="0 0 0"/>
-  </joint>
-  <link name="SurroundingRightLaser_frame"/>
-  <joint name="LaserSensor/Right_projected_sensor_fixedjoint" type="fixed">
-    <parent link="Tibia"/>
-    <child link="SurroundingRightLaser_frame"/>
-    <origin rpy="0 0 -1.75728" xyz="-0.018 -0.0899 -0.334"/>
-    <axis xyz="0 0 0"/>
-  </joint>
-  <link name="HeadTouchFront_frame"/>
-  <joint name="Head/Touch/Front_sensor_fixedjoint" type="fixed">
-    <parent link="Head"/>
-    <child link="HeadTouchFront_frame"/>
-    <origin rpy="0 0.20944 0" xyz="0.028175 0 0.21267"/>
-    <axis xyz="0 0 0"/>
-  </joint>
-  <link name="VerticalRightLaser_frame"/>
-  <joint name="LaserSensor/VerticalRight_sensor_fixedjoint" type="fixed">
-    <parent link="Tibia"/>
-    <child link="VerticalRightLaser_frame"/>
-    <origin rpy="0 0.349066 0" xyz="0.0562 0 -0.0692"/>
-    <axis xyz="0 0 0"/>
-  </joint>
-  <link name="SonarFront_frame"/>
-  <joint name="Sonar/Front_sensor_fixedjoint" type="fixed">
-    <parent link="Tibia"/>
-    <child link="SonarFront_frame"/>
-    <origin rpy="0 -0.322858 0" xyz="0.0699 0 -0.1023"/>
-    <axis xyz="0 0 0"/>
-  </joint>
-  <link name="BumperFL_frame"/>
-  <joint name="Bumper/FrontLeft_sensor_fixedjoint" type="fixed">
-    <parent link="Tibia"/>
-    <child link="BumperFL_frame"/>
-    <origin rpy="0 0 0.48886" xyz="0.129 0.227 -0.264"/>
-    <axis xyz="0 0 0"/>
-  </joint>
-  <link name="CameraBottom_frame"/>
-  <joint name="CameraBottom_sensor_fixedjoint" type="fixed">
-    <parent link="Head"/>
-    <child link="CameraBottom_frame"/>
-    <origin rpy="0 0.698132 0" xyz="0.09262 0 0.06177"/>
-    <axis xyz="0 0 0"/>
-  </joint>
-  <link name="CameraTop_optical_frame"/>
-  <joint name="CameraTop_optical_frame_fixedjoint" type="fixed">
-    <parent link="CameraTop_frame"/>
-    <child link="CameraTop_optical_frame"/>
-    <origin rpy="-1.57079632679 0 -1.57079632679" xyz="0 0 0"/>
-  </joint>
-  <link name="ImuBaseAccelerometer_frame"/>
-  <joint name="AccelerometerBase_sensor_fixedjoint" type="fixed">
-    <parent link="Tibia"/>
-    <child link="ImuBaseAccelerometer_frame"/>
-    <origin rpy="0 0 0" xyz="0.0147 -0.0017 -0.26319"/>
-    <axis xyz="0 0 0"/>
-  </joint>
-  <link name="ImuTorsoGyrometer_frame"/>
-  <joint name="Gyrometer_sensor_fixedjoint" type="fixed">
-    <parent link="torso"/>
-    <child link="ImuTorsoGyrometer_frame"/>
-    <origin rpy="0 0 0" xyz="0.00204 -0.03491 -0.00959"/>
-    <axis xyz="0 0 0"/>
-  </joint>
-  <link name="Tablet_frame"/>
-  <joint name="Tablet_sensor_fixedjoint" type="fixed">
-    <parent link="torso"/>
-    <child link="Tablet_frame"/>
-    <origin rpy="0 -0.523599 0" xyz="0.0839249 0 0.06251"/>
-    <axis xyz="0 0 0"/>
-  </joint>
-  <link name="HeadTouchRear_frame"/>
-  <joint name="Head/Touch/Rear_sensor_fixedjoint" type="fixed">
-    <parent link="Head"/>
-    <child link="HeadTouchRear_frame"/>
-    <origin rpy="0 -0.314159 0" xyz="-0.03376 0 0.21052"/>
-    <axis xyz="0 0 0"/>
-  </joint>
-  <link name="BumperFR_frame"/>
-  <joint name="Bumper/FrontRight_sensor_fixedjoint" type="fixed">
-    <parent link="Tibia"/>
-    <child link="BumperFR_frame"/>
-    <origin rpy="0 0 -0.48886" xyz="0.129 -0.227 -0.264"/>
-    <axis xyz="0 0 0"/>
-  </joint>
-  <link name="SurroundingFrontLaser_frame"/>
-  <joint name="LaserSensor/Front_projected_sensor_fixedjoint" type="fixed">
-    <parent link="Tibia"/>
-    <child link="SurroundingFrontLaser_frame"/>
-    <origin rpy="0 0 0" xyz="0.0562 0 -0.334"/>
-    <axis xyz="0 0 0"/>
-  </joint>
-  <link name="ChestButton_frame"/>
-  <joint name="ChestBoard/Button_sensor_fixedjoint" type="fixed">
-    <parent link="torso"/>
-    <child link="ChestButton_frame"/>
-    <origin rpy="0 0 0" xyz="0.049871 0.001588 0.055163"/>
-    <axis xyz="0 0 0"/>
-  </joint>
-  <link name="HeadTouchMiddle_frame"/>
-  <joint name="Head/Touch/Middle_sensor_fixedjoint" type="fixed">
-    <parent link="Head"/>
-    <child link="HeadTouchMiddle_frame"/>
-    <origin rpy="0 -0.0349066 0" xyz="0.0041 0 0.2159"/>
-    <axis xyz="0 0 0"/>
-  </joint>
+<!--  <link name="SonarBack_frame"/>-->
+<!--  <joint name="Sonar/Back_sensor_fixedjoint" type="fixed">-->
+<!--    <parent link="Tibia"/>-->
+<!--    <child link="SonarBack_frame"/>-->
+<!--    <origin rpy="-1.81761e-08 -0.209438 -3.14159" xyz="-0.0718 0 -0.0534"/>-->
+<!--    <axis xyz="0 0 0"/>-->
+<!--  </joint>-->
+<!--  <link name="CameraBottom_optical_frame"/>-->
+<!--  <joint name="CameraBottom_optical_frame_fixedjoint" type="fixed">-->
+<!--    <parent link="CameraBottom_frame"/>-->
+<!--    <child link="CameraBottom_optical_frame"/>-->
+<!--    <origin rpy="-1.57079632679 0 -1.57079632679" xyz="0 0 0"/>-->
+<!--  </joint>-->
+<!--  <link name="CameraDepth_optical_frame"/>-->
+<!--  <joint name="CameraDepth_optical_frame_fixedjoint" type="fixed">-->
+<!--    <parent link="CameraDepth_frame"/>-->
+<!--    <child link="CameraDepth_optical_frame"/>-->
+<!--    <origin rpy="-1.57079632679 0 -1.57079632679" xyz="0 0 0"/>-->
+<!--  </joint>-->
+<!--  <link name="LHandTouchBack_frame"/>-->
+<!--  <joint name="LHand/Touch/Back_sensor_fixedjoint" type="fixed">-->
+<!--    <parent link="l_wrist"/>-->
+<!--    <child link="LHandTouchBack_frame"/>-->
+<!--    <origin rpy="1.5708 -1.5708 -3.14159" xyz="0.0523 0 0.0304"/>-->
+<!--    <axis xyz="0 0 0"/>-->
+<!--  </joint>-->
+<!--  <link name="VerticalLeftLaser_frame"/>-->
+<!--  <joint name="LaserSensor/VerticalLeft_sensor_fixedjoint" type="fixed">-->
+<!--    <parent link="Tibia"/>-->
+<!--    <child link="VerticalLeftLaser_frame"/>-->
+<!--    <origin rpy="0 0.349066 0" xyz="0.0562 0 -0.0692"/>-->
+<!--    <axis xyz="0 0 0"/>-->
+<!--  </joint>-->
+<!--  <link name="SurroundingFrontLaser_device_frame"/>-->
+<!--  <joint name="LaserSensor/Front_sensor_fixedjoint" type="fixed">-->
+<!--    <parent link="Tibia"/>-->
+<!--    <child link="SurroundingFrontLaser_device_frame"/>-->
+<!--    <origin rpy="0 0.349066 0" xyz="0.0562 0 -0.0692"/>-->
+<!--    <axis xyz="0 0 0"/>-->
+<!--  </joint>-->
+<!--  <link name="BumperB_frame"/>-->
+<!--  <joint name="Bumper/Back_sensor_fixedjoint" type="fixed">-->
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
Commit message: a little bit more stable

File: urdf/pepper.urdf.xacro (robot description, xacro)
@@ -136,5 +136,5 @@
     <parent link="base_link"/>
     <child link="torso"/>
-    <origin rpy="0 0 0" xyz="-0.1 0 0.8"/>
+    <origin rpy="0 0 0" xyz="-0.1 0 0.83"/>
     <axis xyz="0 0 0"/>
   </joint>
