Commit message: pepper can now move (not perfect motion when braking)

File: urdf/pepper.urdf.xacro (robot description, xacro)
@@ -21,10 +21,10 @@
 <!--      <material name="light_black"/>-->
 <!--    </visual>-->
-    <collision>
-      <origin xyz="0 0 0.3" />
-      <geometry>
-        <box size="0.5 0.15 0.2"/>
-      </geometry>
-    </collision>
+<!--    <collision>-->
+<!--      <origin xyz="0 0 0.3" />-->
+<!--      <geometry>-->
+<!--        <box size="0.5 0.15 0.2"/>-->
+<!--      </geometry>-->
+<!--    </collision>-->
     <inertial>
       <origin xyz="0 0 0" rpy="0 0 0"/>
@@ -141,6 +141,6 @@
   <link name="torso">
     <inertial>
-      <mass value="0.001"/>
-      <inertia ixx="0.0" ixy="0" ixz="0.0" iyy="0.0" iyz="-0.0" izz="0.0"/>
+      <mass value="1e-6"/>
+      <inertia ixx="1e-9" ixy="0" ixz="0.0" iyy="1e-9" iyz="-0.0" izz="1e-9"/>
       <origin rpy="0 0 0" xyz="0.00322 0 -0.01029"/>
     </inertial>
@@ -151,10 +151,10 @@
       <origin rpy="0 0 0" xyz="0 0 0"/>
     </visual>
-    <collision>
-      <geometry>
-        <mesh filename="package://pepper_meshes/meshes/1.0/Torso_0.10.stl" scale="0.1 0.1 0.1"/>
-      </geometry>
-      <origin rpy="0 0 0" xyz="0 0 0"/>
-    </collision>
+<!--    <collision>-->
+<!--      <geometry>-->
+<!--        <mesh filename="package://pepper_meshes/meshes/1.0/Torso_0.10.stl" scale="0.1 0.1 0.1"/>-->
+<!--      </geometry>-->
+<!--      <origin rpy="0 0 0" xyz="0 0 0"/>-->
+<!--    </collision>-->
   </link>
   <joint name="HeadYaw" type="fixed">
@@ -167,7 +167,7 @@
   <link name="Neck">
     <inertial>
-      <mass value="0.001"/>
-      <inertia ixx="0.0" ixy="0" ixz="0" iyy="0" iyz="2.09863e-06" izz="0.000215252"/>
-      <origin rpy="0 0 0" xyz="-0.00207 0 -0.02636"/>
+      <mass value="1e-6"/>
+      <inertia ixx="1e-9" ixy="0" ixz="0.0" iyy="1e-9" iyz="-0.0" izz="1e-9"/>
+      <origin rpy="0 0 0" xyz="0.00322 0 -0.01029"/>
     </inertial>
     <visual>
@@ -177,10 +177,10 @@
       <origin rpy="0 0 0" xyz="0 0 0"/>
     </visual>
-    <collision>
-      <geometry>
-        <mesh filename="package://pepper_meshes/meshes/1.0/HeadYaw_0.10.stl" scale="0.1 0.1 0.1"/>
-      </geometry>
-      <origin rpy="0 0 0" xyz="0 0 0"/>
-    </collision>
+<!--    <collision>-->
+<!--      <geometry>-->
+<!--        <mesh filename="package://pepper_meshes/meshes/1.0/HeadYaw_0.10.stl" scale="0.1 0.1 0.1"/>-->
+<!--      </geometry>-->
+<!--      <origin rpy="0 0 0" xyz="0 0 0"/>-->
+<!--    </collision>-->
   </link>
   <joint name="HeadPitch" type="fixed">
@@ -193,7 +193,7 @@
   <link name="Head">
     <inertial>
-      <mass value="1.51893"/>
-      <inertia ixx="0.00597209" ixy="0" ixz="0.000125138" iyy="0.0059054" iyz="4.3428e-07" izz="0.00570374"/>
-      <origin rpy="0 0 0" xyz="0.00312 0 0.11152"/>
+      <mass value="1e-6"/>
+      <inertia ixx="1e-9" ixy="0" ixz="0.0" iyy="1e-9" iyz="-0.0" izz="1e-9"/>
+      <origin rpy="0 0 0" xyz="0.00322 0 -0.01029"/>
     </inertial>
     <visual>
@@ -203,10 +203,10 @@
       <origin rpy="0 0 0" xyz="0 0 0"/>
     </visual>
-    <collision>
-      <geometry>
-        <mesh filename="package://pepper_meshes/meshes/1.0/HeadPitch_0.10.stl" scale="0.1 0.1 0.1"/>
-      </geometry>
-      <origin rpy="0 0 0" xyz="0 0 0"/>
-    </collision>
+<!--    <collision>-->
+<!--      <geometry>-->
+<!--        <mesh filename="package://pepper_meshes/meshes/1.0/HeadPitch_0.10.stl" scale="0.1 0.1 0.1"/>-->
+<!--      </geometry>-->
+<!--      <origin rpy="0 0 0" xyz="0 0 0"/>-->
+<!--    </collision>-->
   </link>
   <joint name="HipRoll" type="fixed">
@@ -219,7 +219,7 @@
   <link name="Hip">
     <inertial>
-      <mass value="1.02338"/>
-      <inertia ixx="0.00502422" ixy="0" ixz="-2.54911e-05" iyy="0.00640971" iyz="0.000159449" izz="0.00441082"/>
-      <origin rpy="0 0 0" xyz="0.00032 0 -0.06039"/>
+      <mass value="1e-6"/>
+      <inertia ixx="1e-9" ixy="0" ixz="0.0" iyy="1e-9" iyz="-0.0" izz="1e-9"/>
+      <origin rpy="0 0 0" xyz="0.00322 0 -0.01029"/>
     </inertial>
     <visual>
@@ -229,10 +229,10 @@
       <origin rpy="0 0 0" xyz="0 0 0"/>
     </visual>
-    <collision>
-      <geometry>
-        <mesh filename="package://pepper_meshes/meshes/1.0/HipRoll_0.10.stl" scale="0.1 0.1 0.1"/>
-      </geometry>
-      <origin rpy="0 0 0" xyz="0 0 0"/>
-    </collision>
+<!--    <collision>-->
+<!--      <geometry>-->
+<!--        <mesh filename="package://pepper_meshes/meshes/1.0/HipRoll_0.10.stl" scale="0.1 0.1 0.1"/>-->
+<!--      </geometry>-->
+<!--      <origin rpy="0 0 0" xyz="0 0 0"/>-->
+<!--    </collision>-->
   </link>
   <joint name="HipPitch" type="fixed">
@@ -245,7 +245,7 @@
   <link name="Pelvis">
     <inertial>
-      <mass value="2.45917"/>
-      <inertia ixx="0.034351" ixy="0" ixz="0.000223034" iyy="0.0303122" iyz="-8.37542e-05" izz="0.0143771"/>
-      <origin rpy="0 0 0" xyz="0.00237 0 -0.09654"/>
+      <mass value="1e-6"/>
+      <inertia ixx="1e-9" ixy="0" ixz="0.0" iyy="1e-9" iyz="-0.0" izz="1e-9"/>
+      <origin rpy="0 0 0" xyz="0.00322 0 -0.01029"/>
     </inertial>
     <visual>
@@ -255,10 +255,10 @@
       <origin rpy="0 0 0" xyz="0 0 0"/>
     </visual>
-    <collision>
-      <geometry>
-        <mesh filename="package://pepper_meshes/meshes/1.0/HipPitch_0.10.stl" scale="0.1 0.1 0.1"/>
-      </geometry>
-      <origin rpy="0 0 0" xyz="0 0 0"/>
-    </collision>
+<!--    <collision>-->
+<!--      <geometry>-->
+<!--        <mesh filename="package://pepper_meshes/meshes/1.0/HipPitch_0.10.stl" scale="0.1 0.1 0.1"/>-->
+<!--      </geometry>-->
+<!--      <origin rpy="0 0 0" xyz="0 0 0"/>-->
+<!--    </collision>-->
   </link>
   <joint name="KneePitch" type="fixed">
@@ -271,7 +271,7 @@
   <link name="Tibia">
     <inertial>
-      <mass value="11.6015"/>
-      <inertia ixx="0.129229" ixy="-0.000401943" ixz="0.00048556" iyy="0.122839" iyz="-1.01666e-08" izz="0.108168"/>
-      <origin rpy="0 0 0" xyz="0.00220451 0 -0.185729"/>
+      <mass value="1e-6"/>
+      <inertia ixx="1e-9" ixy="0" ixz="0.0" iyy="1e-9" iyz="-0.0" izz="1e-9"/>
+      <origin rpy="0 0 0" xyz="0.00322 0 -0.01029"/>
     </inertial>
     <visual>
@@ -281,10 +281,10 @@
       <origin rpy="0 0 0" xyz="0 0 0"/>
     </visual>
-    <collision>
-      <geometry>
-        <mesh filename="package://pepper_meshes/meshes/1.0/KneePitch_0.10.stl" scale="0.1 0.1 0.1"/>
-      </geometry>
-      <origin rpy="0 0 0" xyz="0 0 0"/>
-    </collision>
+<!--    <collision>-->
+<!--      <geometry>-->
+<!--        <mesh filename="package://pepper_meshes/meshes/1.0/KneePitch_0.10.stl" scale="0.1 0.1 0.1"/>-->
+<!--      </geometry>-->
+<!--      <origin rpy="0 0 0" xyz="0 0 0"/>-->
+<!--    </collision>-->
   </link>
 <!--  <joint name="base_footprint_joint" type="fixed">-->
@@ -303,7 +303,7 @@
   <link name="LShoulder">
     <inertial>
-      <mass value="0.3125"/>
-      <inertia ixx="0.000361198" ixy="-1.98347e-06" ixz="6.35907e-07" iyy="0.000137229" iyz="-5.68878e-06" izz="0.000399194"/>
-      <origin rpy="0 0 0" xyz="0.00018 -0.01856 0.00099"/>
+      <mass value="1e-6"/>
+      <inertia ixx="1e-9" ixy="0" ixz="0.0" iyy="1e-9" iyz="-0.0" izz="1e-9"/>
+      <origin rpy="0 0 0" xyz="0.00322 0 -0.01029"/>
     </inertial>
     <visual>
@@ -313,10 +313,10 @@
       <origin rpy="0 0 0" xyz="0 0 0"/>
     </visual>
-    <collision>
-      <geometry>
-        <mesh filename="package://pepper_meshes/meshes/1.0/LShoulderPitch_0.10.stl" scale="0.1 0.1 0.1"/>
-      </geometry>
-      <origin rpy="0 0 0" xyz="0 0 0"/>
-    </collision>
+<!--    <collision>-->
+<!--      <geometry>-->
+<!--        <mesh filename="package://pepper_meshes/meshes/1.0/LShoulderPitch_0.10.stl" scale="0.1 0.1 0.1"/>-->
+<!--      </geometry>-->
+<!--      <origin rpy="0 0 0" xyz="0 0 0"/>-->
+<!--    </collision>-->
   </link>
   <joint name="LShoulderRoll" type="fixed">
@@ -329,6 +329,6 @@
   <link name="LBicep">
     <inertial>
-      <mass value="0.50527"/>
-      <inertia ixx="0.000500872" ixy="-3.55918e-05" ixz="8.51263e-05" iyy="0.00126284" iyz="9.06813e-06" izz="0.00115718"/>
+      <mass value="1e-6"/>
+      <inertia ixx="1e-9" ixy="0" ixz="0.0" iyy="1e-9" iyz="-0.0" izz="1e-9"/>
       <origin rpy="0 0 0" xyz="0.08151 0.01284 -0.01017"/>
     </inertial>
@@ -339,10 +339,10 @@
       <origin rpy="0 0 0" xyz="0 0 0"/>
     </visual>
-    <collision>
-      <geometry>
-        <mesh filename="package://pepper_meshes/meshes/1.0/LShoulderRoll_0.10.stl" scale="0.1 0.1 0.1"/>
-      </geometry>
-      <origin rpy="0 0 0" xyz="0 0 0"/>
-    </collision>
+<!--    <collision>-->
+<!--      <geometry>-->
+<!--        <mesh filename="package://pepper_meshes/meshes/1.0/LShoulderRoll_0.10.stl" scale="0.1 0.1 0.1"/>-->
+<!--      </geometry>-->
+<!--      <origin rpy="0 0 0" xyz="0 0 0"/>-->
+<!--    </collision>-->
   </link>
   <joint name="LElbowYaw" type="fixed">
@@ -355,6 +355,6 @@
   <link name="LElbow">
     <inertial>
-      <mass value="0.27495"/>
-      <inertia ixx="0.000122971" ixy="9.86024e-07" ixz="-2.55838e-05" iyy="0.000331766" iyz="-1.98925e-06" izz="0.000303047"/>
+      <mass value="1e-6"/>
+      <inertia ixx="1e-9" ixy="0" ixz="0.0" iyy="1e-9" iyz="-0.0" izz="1e-9"/>
       <origin rpy="0 0 0" xyz="-0.02297 -0.00019 0.00119"/>
     </inertial>
@@ -365,10 +365,10 @@
       <origin rpy="0 0 0" xyz="0 0 0"/>
     </visual>
-    <collision>
-      <geometry>
-        <mesh filename="package://pepper_meshes/meshes/1.0/LElbowYaw_0.10.stl" scale="0.1 0.1 0.1"/>
-      </geometry>
-      <origin rpy="0 0 0" xyz="0 0 0"/>
-    </collision>
+<!--    <collision>-->
+<!--      <geometry>-->
+<!--        <mesh filename="package://pepper_meshes/meshes/1.0/LElbowYaw_0.10.stl" scale="0.1 0.1 0.1"/>-->
+<!--      </geometry>-->
+<!--      <origin rpy="0 0 0" xyz="0 0 0"/>-->
+<!--    </collision>-->
   </link>
   <joint name="LElbowRoll" type="fixed">
@@ -381,6 +381,6 @@
   <link name="LForeArm">
     <inertial>
-      <mass value="0.16579"/>
-      <inertia ixx="0.00156513" ixy="1.47517e-05" ixz="-6.05746e-05" iyy="0.00173219" iyz="-1.7619e-07" izz="0.000273081"/>
+      <mass value="1e-6"/>
+      <inertia ixx="1e-9" ixy="0" ixz="0.0" iyy="1e-9" iyz="-0.0" izz="1e-9"/>
       <origin rpy="0 0 0" xyz="0.0593 0.00271 -0.01014"/>
     </inertial>
@@ -391,10 +391,10 @@
       <origin rpy="0 0 0" xyz="0 0 0"/>
     </visual>
-    <collision>
-      <geometry>
-        <mesh filename="package://pepper_meshes/meshes/1.0/LElbowRoll_0.10.stl" scale="0.1 0.1 0.1"/>
-      </geometry>
-      <origin rpy="0 0 0" xyz="0 0 0"/>
-    </collision>
+<!--    <collision>-->
+<!--      <geometry>-->
+<!--        <mesh filename="package://pepper_meshes/meshes/1.0/LElbowRoll_0.10.stl" scale="0.1 0.1 0.1"/>-->
+<!--      </geometry>-->
+<!--      <origin rpy="0 0 0" xyz="0 0 0"/>-->
+<!--    </collision>-->
   </link>
   <joint name="LWristYaw" type="fixed">
@@ -407,6 +407,6 @@
   <link name="l_wrist">
     <inertial>
-      <mass value="0.27555"/>
-      <inertia ixx="0.000151643" ixy="1.06629e-05" ixz="2.89509e-06" iyy="0.000431099" iyz="-3.13715e-06" izz="0.000456172"/>
+      <mass value="1e-6"/>
+      <inertia ixx="1e-9" ixy="0" ixz="0.0" iyy="1e-9" iyz="-0.0" izz="1e-9"/>
       <origin rpy="0 0 0" xyz="0.03536 -0.00072 -0.00207"/>
     </inertial>
@@ -433,6 +433,6 @@
   <link name="l_gripper">
     <inertial>
-      <mass value="2e-06"/>
-      <inertia ixx="1.1e-09" ixy="0" ixz="0" iyy="1.1e-09" iyz="0" izz="1.1e-09"/>
+      <mass value="1e-6"/>
+      <inertia ixx="1e-9" ixy="0" ixz="0.0" iyy="1e-9" iyz="-0.0" izz="1e-9"/>
     </inertial>
   </link>
@@ -446,6 +446,6 @@
   <link name="RShoulder">
     <inertial>
-      <mass value="0.3125"/>
-      <inertia ixx="0.000361198" ixy="1.98347e-06" ixz="6.35907e-07" iyy="0.000137229" iyz="5.68878e-06" izz="0.000399194"/>
+      <mass value="1e-6"/>
+      <inertia ixx="1e-9" ixy="0" ixz="0.0" iyy="1e-9" iyz="-0.0" izz="1e-9"/>
       <origin rpy="0 0 0" xyz="0.00018 0.01856 0.00099"/>
     </inertial>
@@ -472,6 +472,6 @@
   <link name="RBicep">
     <inertial>
-      <mass value="0.50527"/>
-      <inertia ixx="0.000500872" ixy="3.55918e-05" ixz="8.51263e-05" iyy="0.00126284" iyz="-9.06813e-06" izz="0.00115718"/>
+      <mass value="1e-6"/>
+      <inertia ixx="1e-9" ixy="0" ixz="0.0" iyy="1e-9" iyz="-0.0" izz="1e-9"/>
       <origin rpy="0 0 0" xyz="0.08151 -0.01284 -0.01017"/>
     </inertial>
@@ -498,6 +498,6 @@
   <link name="RElbow">
     <inertial>
-      <mass value="0.27495"/>
-      <inertia ixx="0.000122971" ixy="-9.86024e-07" ixz="-2.55838e-05" iyy="0.000331766" iyz="1.98925e-06" izz="0.000303047"/>
+      <mass value="1e-6"/>
+      <inertia ixx="1e-9" ixy="0" ixz="0.0" iyy="1e-9" iyz="-0.0" izz="1e-9"/>
       <origin rpy="0 0 0" xyz="-0.02297 0.00019 0.00119"/>
     </inertial>
@@ -508,10 +508,10 @@
       <origin rpy="0 0 0" xyz="0 0 0"/>
     </visual>
-    <collision>
-      <geometry>
-        <mesh filename="package://pepper_meshes/meshes/1.0/RElbowYaw_0.10.stl" scale="0.1 0.1 0.1"/>
-      </geometry>
-      <origin rpy="0 0 0" xyz="0 0 0"/>
-    </collision>
+<!--    <collision>-->
+<!--      <geometry>-->
+<!--        <mesh filename="package://pepper_meshes/meshes/1.0/RElbowYaw_0.10.stl" scale="0.1 0.1 0.1"/>-->
+<!--      </geometry>-->
+<!--      <origin rpy="0 0 0" xyz="0 0 0"/>-->
+<!--    </collision>-->
   </link>
   <joint name="RElbowRoll" type="fixed">
@@ -524,6 +524,6 @@
   <link name="RForeArm">
     <inertial>
-      <mass value="0.16579"/>
-      <inertia ixx="0.00156513" ixy="-1.47517e-05" ixz="-6.05746e-05" iyy="0.00173219" iyz="1.7619e-07" izz="0.000273081"/>
+      <mass value="1e-6"/>
+      <inertia ixx="1e-9" ixy="0" ixz="0.0" iyy="1e-9" iyz="-0.0" izz="1e-9"/>
       <origin rpy="0 0 0" xyz="0.0593 -0.00271 -0.01014"/>
     </inertial>
@@ -550,6 +550,6 @@
   <link name="r_wrist">
     <inertial>
-      <mass value="0.27555"/>
-      <inertia ixx="0.000151643" ixy="-1.06629e-05" ixz="2.89509e-06" iyy="0.000431099" iyz="3.13715e-06" izz="0.000456172"/>
+      <mass value="1e-6"/>
+      <inertia ixx="1e-9" ixy="0" ixz="0.0" iyy="1e-9" iyz="-0.0" izz="1e-9"/>
       <origin rpy="0 0 0" xyz="0.03536 0.00072 -0.00207"/>
     </inertial>
@@ -576,6 +576,6 @@
   <link name="r_gripper">
     <inertial>
-      <mass value="2e-06"/>
-      <inertia ixx="1.1e-09" ixy="0" ixz="0" iyy="1.1e-09" iyz="0" izz="1.1e-09"/>
+      <mass value="1e-6"/>
+      <inertia ixx="1e-9" ixy="0" ixz="0.0" iyy="1e-9" iyz="-0.0" izz="1e-9"/>
     </inertial>
   </link>
@@ -803,6 +803,6 @@
   <link name="RFinger41_link">
     <inertial>
-      <mass value="2e-06"/>
-      <inertia ixx="1.1e-09" ixy="0" ixz="0" iyy="1.1e-09" iyz="0" izz="1.1e-09"/>
+      <mass value="1e-6"/>
+      <inertia ixx="1e-9" ixy="0" ixz="0.0" iyy="1e-9" iyz="-0.0" izz="1e-9"/>
     </inertial>
     <visual>
@@ -812,10 +812,10 @@
       <origin rpy="0 0 0" xyz="0 0 0"/>
     </visual>
-    <collision>
-      <geometry>
-        <mesh filename="package://pepper_meshes/meshes/1.0/RFinger41_0.10.stl" scale="0.1 0.1 0.1"/>
-      </geometry>
-      <origin rpy="0 0 0" xyz="0 0 0"/>
-    </collision>
+<!--    <collision>-->
+<!--      <geometry>-->
+<!--        <mesh filename="package://pepper_meshes/meshes/1.0/RFinger41_0.10.stl" scale="0.1 0.1 0.1"/>-->
+<!--      </geometry>-->
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
Commit message: Fix DepthCamera on Pepper

File: urdf/pepper.urdf.xacro (robot description, xacro)
@@ -14,17 +14,4 @@
   </joint>
   <link name="base_link">
-<!--    <visual>-->
-<!--      <origin xyz="-0.064 0 0.45" rpy="0 0 0"/>-->
-<!--      <geometry>-->
-<!--        <box size="0.23 0.23 0.8" />-->
-<!--      </geometry>-->
-<!--      <material name="light_black"/>-->
-<!--    </visual>-->
-<!--    <collision>-->
-<!--      <origin xyz="0 0 0.3" />-->
-<!--      <geometry>-->
-<!--        <box size="0.5 0.15 0.2"/>-->
-<!--      </geometry>-->
-<!--    </collision>-->
     <inertial>
       <origin xyz="0 0 0" rpy="0 0 0"/>
@@ -35,4 +22,33 @@
     </inertial>
   </link>
+  <joint name="camera_joint" type="fixed">
+    <origin xyz="-0.05 -0.065 1.16" rpy="0 0 0"/>
+    <parent link="base_link"/>
+    <child link="camera_link"/>
+  </joint>
+  <link name="camera_link">
+    <visual>
+     <origin xyz="0 0 0" rpy="1.57 0 1.57"/>
+      <geometry>
+       <mesh filename="package://turtlebot3_description/meshes/sensors/r200.dae" />
+      </geometry>
+    </visual>
+    <collision>
+      <origin xyz="0.003 0.065 0.007" rpy="0 0 0"/>
+      <geometry>
+        <box size="0.012 0.132 0.020"/>
+      </geometry>
+    </collision>
+   <inertial>
+      <mass value="1e-6"/>
+      <inertia ixx="1e-9" ixy="0" ixz="0.0" iyy="1e-9" iyz="-0.0" izz="1e-9"/>
+   </inertial>
+  </link>
+  <joint name="camera_rgb_joint" type="fixed">
+    <origin xyz="0 0 0" rpy="0 0 0"/>
+    <parent link="camera_link"/>
+    <child link="camera_rgb_frame"/>
+  </joint>
+  <link name="camera_rgb_frame"/>
 <!-- Links From Turtle -->
   <joint name="wheel_left_joint" type="continuous">

Commit message: minor changes

File: urdf/pepper.urdf.xacro (robot description, xacro)
@@ -22,4 +22,10 @@
     </inertial>
   </link>
+  <joint name="imu_joint" type="fixed">
+    <parent link="base_link"/>
+    <child link="imu_link"/>
+    <origin xyz="0.0 0 0.068" rpy="0 0 0"/>
+  </joint>
+  <link name="imu_link"/>
   <joint name="camera_joint" type="fixed">
     <origin xyz="-0.05 -0.065 1.16" rpy="0 0 0"/>

Commit message: Commit Last changes on Optical Flow based Legibility

File: urdf/pepper.urdf.xacro (robot description, xacro)
@@ -38,4 +38,5 @@
       <geometry>
        <mesh filename="package://turtlebot3_description/meshes/sensors/r200.dae" />
+<!--       <mesh filename="/home/javad/workspace/catkin_ws/src/gazebo-realsense/models/realsense_camera/meshes/realsense.dae" />-->
       </geometry>
     </visual>

Commit message: Fixed Pepper motion in Gazebo (no slipping!)

File: urdf/pepper.urdf.xacro (robot description, xacro)
@@ -1,6 +1,4 @@
 <?xml version="1.0" ?>
-<robot name="turtlebot3_pepper_v" xmlns:xacro="http://ros.org/wiki/xacro">
-  <xacro:include filename="$(find turtlebot3_description)/urdf/common_properties.xacro"/>
-  <xacro:include filename="$(find turtlebot3_description)/urdf/turtlebot3_waffle.gazebo.xacro"/>
+<robot name="pepper_modified" xmlns:xacro="http://ros.org/wiki/xacro">
   <xacro:property name="r200_cam_rgb_px" value="0.005"/>
   <xacro:property name="r200_cam_rgb_py" value="0.018"/>
@@ -58,5 +56,20 @@
   </joint>
   <link name="camera_rgb_frame"/>
-<!-- Links From Turtle -->
+  <gazebo>
+    <plugin filename="libgazebo_ros_diff_drive.so" name="differential_drive_controller">
+      <alwaysOn>true</alwaysOn>
+      <updateRate>20</updateRate>
+      <leftJoint>wheel_left_joint</leftJoint>
+      <rightJoint>wheel_right_joint</rightJoint>
+      <wheelSeparation>0.4</wheelSeparation>
+      <wheelDiameter>0.2</wheelDiameter>
+      <torque>0.1</torque>
+      <commandTopic>cmd_vel</commandTopic>
+      <odometryTopic>odom</odometryTopic>
+      <odometryFrame>odom</odometryFrame>
+      <robotBaseFrame>base_link</robotBaseFrame>
+    </plugin>
+  </gazebo>
+<!-- Links from Turtlebot -->
   <joint name="wheel_left_joint" type="continuous">
     <parent link="base_link"/>
@@ -66,11 +79,10 @@
   </joint>
   <link name="wheel_left_link">
-    <visual>
-      <origin xyz="0 0 0" rpy="1.57 0 0"/>
-      <geometry>
-        <mesh filename="package://turtlebot3_description/meshes/wheels/left_tire.stl" scale="0.001 0.001 0.001"/>
-      </geometry>
-      <material name="dark"/>
-    </visual>
+<!--    <visual>-->
+<!--      <origin xyz="0 0 0" rpy="1.57 0 0"/>-->
+<!--      <geometry>-->
+<!--      </geometry>-->
+<!--      <material name="dark"/>-->
+<!--    </visual>-->
     <collision>
       <origin xyz="0 0 0" rpy="0 0 0"/>
@@ -94,11 +106,10 @@
   </joint>
   <link name="wheel_right_link">
-    <visual>
-      <origin xyz="0 0 0" rpy="1.57 0 0"/>
-      <geometry>
-        <mesh filename="package://turtlebot3_description/meshes/wheels/right_tire.stl" scale="0.001 0.001 0.001"/>
-      </geometry>
-      <material name="dark"/>
-    </visual>
+<!--    <visual>-->
+<!--      <origin xyz="0 0 0" rpy="1.57 0 0"/>-->
+<!--      <geometry>-->
+<!--      </geometry>-->
+<!--      <material name="dark"/>-->
+<!--    </visual>-->
     <collision>
       <origin xyz="0 0 0" rpy="0 0 0"/>
@@ -159,5 +170,5 @@
     <parent link="base_link"/>
     <child link="torso"/>
-    <origin rpy="0 0 0" xyz="-0.1 0 0.83"/>
+    <origin rpy="0 0 0" xyz="-0.1 0 0.86"/>
     <axis xyz="0 0 0"/>
   </joint>

Commit message: Sim: Improve Pepper motion (smoother)

File: urdf/pepper.urdf.xacro (robot description, xacro)
@@ -167,4 +167,45 @@
   </link>
 <!---->
+  <joint name="caster_front_right_joint" type="fixed">
+    <parent link="base_link"/>
+    <child link="caster_front_right_link"/>
+    <origin xyz="0.1 -0.064 -0.004" rpy="-1.57 0 0"/>
+  </joint>
+  <link name="caster_front_right_link">
+    <collision>
+      <origin xyz="0 0.001 0" rpy="0 0 0"/>
+      <geometry>
+        <box size="0.030 0.009 0.020"/>
+      </geometry>
+    </collision>
+    <inertial>
+      <origin xyz="0 0 0" />
+      <mass value="0.005" />
+      <inertia ixx="0.001" ixy="0.0" ixz="0.0"
+               iyy="0.001" iyz="0.0"
+               izz="0.001" />
+    </inertial>
+  </link>
+  <joint name="caster_front_left_joint" type="fixed">
+    <parent link="base_link"/>
+    <child link="caster_front_left_link"/>
+    <origin xyz="+0.1 0.064 -0.004" rpy="-1.57 0 0"/>
+  </joint>
+  <link name="caster_front_left_link">
+    <collision>
+      <origin xyz="0 0.001 0" rpy="0 0 0"/>
+      <geometry>
+        <box size="0.030 0.009 0.020"/>
+      </geometry>
+    </collision>
+    <inertial>
+      <origin xyz="0 0 0" />
+      <mass value="0.005" />
+      <inertia ixx="0.001" ixy="0.0" ixz="0.0"
+               iyy="0.001" iyz="0.0"
+               izz="0.001" />
+    </inertial>
+  </link>
+<!--  -->
   <joint name="base_link_fixedjoint" type="fixed">
     <parent link="base_link"/>
