Commit message: Add an observer person to the scene (with Camera)

File: urdf/observer.urdf (robot description, URDF)
Before this commit: robot observer_person_d, 2 links, 1 joints
Links:
- link base_link: mass None -> 1.0; geometry collision box size=0.5 0.15 1.8; visual mesh filename=/home/javad/.gazebo/models/person_standing/meshes/standing.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
- link camera_link: mass None -> 0.2; geometry collision box size=0.02 0.02 0.02
Joints:
- joint camera_joint: origin (none) -> xyz=0.045 -0.15 1.78 rpy=0 0.4 -1.57

Commit message: Gazebo: fixed unwanted motion of the observer in the simulator

File: urdf/observer.urdf (robot description, URDF)
Before this commit: robot observer_person_d, 2 links, 1 joints
Links:
- link camera_link: mass 0.2 -> None

Commit message: Sim: Pepper with a bottle of champaign + round tables

File: urdf/observer.urdf (robot description, URDF)
Before this commit: robot observer_person_d, 2 links, 1 joints
Links:
- link base_link: geometry collision box size=0.5 0.15 1.8; visual mesh filename=package://legibot/models/person_standing/meshes/standing.dae

File: urdf/pepper.urdf.xacro (robot description, xacro)
@@ -372,5 +372,5 @@
     <parent link="LBicep"/>
     <child link="LElbow"/>
-    <origin rpy="0 -0.157079 0" xyz="0.1812 0.015 0.00013"/>
+    <origin rpy="-1 -0.157079 0" xyz="0.1812 0.015 0.00013"/>
     <axis xyz="1.0 0 0"/>
     <limit effort="5.428" lower="-2.08567" upper="2.08567" velocity="7.33998"/>
@@ -515,5 +515,5 @@
     <parent link="RBicep"/>
     <child link="RElbow"/>
-    <origin rpy="0 -0.157079 0" xyz="0.1812 -0.015 0.00013"/>
+    <origin rpy="1.25 -0.157079 0" xyz="0.1812 -0.015 0.00013"/>
     <axis xyz="1.0 0 0"/>
     <limit effort="5.428" lower="-2.08567" upper="2.08567" velocity="7.33998"/>
@@ -1374,4 +1374,31 @@
     <mimic joint="RHand" multiplier="0.872665" offset="0"/>
   </joint>
+  <joint name="RBottleInHand" type="fixed">
+    <parent link="r_wrist"/>
+    <child link="wine_bottle_link"/>
+<!--    <axis xyz="0 0 1.0"/>-->
+    <origin rpy="0.2 0 0" xyz="0.07 -0.20 -0.055"/>
+  </joint>
+  <link name="wine_bottle_link">
+    <inertial>
+      <mass value="2e-06"/>
+      <inertia ixx="1e-9" ixy="0" ixz="0.0" iyy="1e-9" iyz="-0.0" izz="1e-9"/>
+    </inertial>
+    <collision>
+      <origin rpy="0 0 0" xyz="0 0 0"/>
+      <geometry>
+          <cylinder>
+              <radius>0.04</radius>
+              <length>0.30</length>
+            </cylinder>
+        </geometry>
+    </collision>
+    <visual>
+      <origin rpy="0 0 0" xyz="0 0 0"/>
+      <geometry>
+        <mesh filename="package://legibot/models/wine_bottle/meshes/bottle.dae" scale="0.02 0.02 0.02"/>
+      </geometry>
+    </visual>
+  </link>
   <link name="LFinger31_link">
     <inertial>

Commit message: minor fixes

File: urdf/observer.urdf (robot description, URDF)
Before this commit: robot observer_person_d, 2 links, 1 joints
Joints:
- joint camera_joint: origin xyz=0.045 -0.15 1.78 rpy=0 0.4 -1.57 -> xyz=0.045 0.35 2.18 rpy=0 0.6 -1.57
